File: hardware/monitor.kicad_pcb (KiCad board)
At the start: 2 copper layers, 55.9 x 64.8 mm, 52 parts, among them J1 CT, J10 Spare, J2 T1, J3 RPi Interconnect, J5 Pulse, J6 ISP, J7 UART, J8 Whip antenna, J9 SMA antenna, SW1 Reset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

Commit message: Hardware revision 2
Parts:
- moved J7 4.07 mm to (102.9, 73.7)
- moved C5 1.27 mm to (87.6, 71.8)
Routing:
- net Net-(C4-Pad1): track 17.0 -> 37.5 mm
- net /Microcontroller/RF_SS: track 59.2 -> 52.6 mm
- net Net-(C11-Pad1): track 8.06 -> 12.0 mm
- net /Microcontroller/Reset: track 85.7 -> 82.7 mm
- net /Microcontroller/RX: track 49.0 -> 50.5 mm
- net /Microcontroller/RF_IRQ: track 34.1 -> 33.3 mm
Other:
- board text added: "Assembled"
- board text added: "Taransay Monitor r2 2020-08-13 Sean Leavey Based on EmonTx/EmonTH by OpenEnergyMonitor"
- board text removed: "Assembler"
- board text removed: "Date"
- board text removed: "Taransay Monitor r1 2018-09-29 Sean Leavey Based on EmonTx/EmonTH by OpenEnergyMonitor"
