File: hardware/switch/switch.kicad_pcb (KiCad board)
At the start: 2 copper layers, 96.5 x 49.5 mm, 33 parts, among them J1 Power, J2 DC, J3 External button 1, J4 External button 2, J5 Analog, J6 Digital, J7 Analog breakout, J8 Digital breakout, K1 FINDER-32.21-x000, K2 FINDER-32.21-x000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

Commit message: Remove JLCPCB silkscreen text
Other:
- board text removed: "JLCJLCJLCJLC"
