File: hardware/taransay/taransay.kicad_pcb (KiCad board)
At the start: 2 copper layers, 31.8 x 39.4 mm, 33 parts, among them J1 VIN, J2 Analog, J3 Digital, J4 Whip antenna, J5 SMA antenna, J6 ISP, J7 UART, J8 RPi Interconnect, U1 LTC3525-3.3, U2 LM3480-3.3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

Commit message: Update Taransay board to Kicad 6
Connections:
- net /~RST renamed /~{RST}
Other:
- net class Default removed
- net class Power removed
- net class RF removed
- net class Spare removed
- board text added: "~{RST}"
- board text removed: "~RST"
